Commit message: charge to controller

File: camera_stereo/urdf/myCameraStereo.urdf (robot description, URDF)
Before this commit: robot myCameraStereo, 1 links, 0 joints
Links:
- added link second_link, mass 1000; collision box size=0.005 0.005 0.015; visual box size=0.05 0.05 0.15
- added link world
- link cameras: mass 1 -> 0.1; geometry collision box size=0.05 0.05 0.05; visual mesh filename=file://$(find camera_stereo)/meshes/ZEDM.stl scale=1 1 1
Joints:
- added joint base_to_second_joint: type prismatic, parent second_link, child cameras, origin xyz=0.3 0. 0 rpy=0.0 0.0 0.0, axis 1 0 0, limit lower=-1 upper=5 effort=10000 velocity=1
- added joint fixed_joint: type revolute, parent world, child second_link, origin xyz=0 0 0 rpy=0 0 0, axis 0 0 1, limit lower=0 upper=0 effort=1000000000 velocity=0

File: turtlebot3/turtlebot3_description/urdf/turtlebot3_burger_for_autorace.gazebo.xacro (robot description, xacro)
@@ -126,5 +126,64 @@
   <!--link : https://www.raspberrypi.org/documentation/hardware/camera/-->
   <gazebo reference="camera_rgb_frame">
-    <sensor type="camera" name="Pi Camera">
+  <sensor type="multicamera" name="stereo_camera">
+      <update_rate>30</update_rate>
+        <camera name="left">
+          <horizontal_fov>1.3962634</horizontal_fov>
+          <image>
+            <width>640</width>
+            <height>480</height>
+            <format>R8G8B8</format>
+          </image>
+          <clip>
+            <near>0.02</near>
+            <far>300</far>
+          </clip>
+          <noise>
+            <type>gaussian</type>
+            <mean>0.0</mean>
+            <stddev>0.007</stddev>
+          </noise>
+        </camera>
+        <camera name="right">
+          <pose>0 -0.10 0 0 0 0</pose>
+          <horizontal_fov>1.3962634</horizontal_fov>
+          <image>
+            <width>640</width>
+            <height>480</height>
+            <format>R8G8B8</format>
+          </image>
+          <clip>
+            <near>0.02</near>
+            <far>300</far>
+          </clip>
+          <noise>
+            <type>gaussian</type>
+            <mean>0.0</mean>
+            <stddev>0.007</stddev>
+          </noise>
+        </camera>
+      <plugin name="camera_controller" filename="libgazebo_ros_multicamera.so">
+        <updateRate>0.0</updateRate>
+        <scale_to_hfov>true</scale_to_hfov>
+        <alwaysOn>true</alwaysOn>
+        <baseline>0.12</baseline>
+        <frameName>camera_rgb_optical_frame</frameName>
+        <cameraName>myCameraStereo/stereo_camera</cameraName>
+        <cameraInfoTopicName>camera_info</cameraInfoTopicName>
+        <hackBaseline>0.07</hackBaseline>
+        <focal_length>320</focal_length>
+        <distortion_k1>0.00000001</distortion_k1>
+        <distortion_k2>0.00000001</distortion_k2>
+        <distortion_k3>0.00000001</distortion_k3>
+        <distortion_t1>0.00000001</distortion_t1>
+        <distortion_t2>0.00000001</distortion_t2>
+        <!-- required for ros depth cam -->
+        <imageTopicName>image_raw</imageTopicName>
+        <pointCloudTopicName>camera_cloud</pointCloudTopicName>
+        <depthImageTopicName>camera_depth</depthImageTopicName>
+        <depthImageCameraInfoTopicName>depth_info</depthImageCameraInfoTopicName>
+      </plugin>
+    </sensor>
+    <!-- <sensor type="camera" name="Pi Camera">
       <always_on>true</always_on>
       <visualize>$(arg camera_visual)</visualize>
@@ -155,5 +214,5 @@
         <distortionT2>0.0</distortionT2>
       </plugin>
-    </sensor>
+    </sensor> -->
   </gazebo>
 </robot>

Commit message: Modification to adapt to orb slam2

File: camera_stereo/urdf/myCameraStereo.urdf (robot description, URDF)
Before this commit: robot myCameraStereo, 3 links, 2 joints
Links:
- added link third_link, mass 1000; collision box size=0.005 0.005 0.015; visual sphere radius=0.05
- link cameras: mass 0.1 -> 0.5
- link second_link: mass 1000 -> 1; geometry collision box size=0.005 0.005 0.015; visual sphere radius=0.05
Joints:
- added joint base_to_third_joint: type prismatic, parent third_link, child second_link, origin xyz=0 0 0.1 rpy=0.0 0.0 0.0, axis 1 0 0, limit lower=-1 upper=5 effort=100 velocity=1
- joint base_to_second_joint: axis 1 0 0 -> 0 1 0; limit lower=-1 upper=5 effort=10000 velocity=1 -> lower=-1 upper=5 effort=100 velocity=1; origin xyz=0.3 0. 0 rpy=0.0 0.0 0.0 -> xyz=0 0 0.6 rpy=0.0 0.0 ${pi/2}
- joint fixed_joint: axis 0 0 1 -> 0 0 0; child second_link -> third_link; limit lower=0 upper=0 effort=1000000000 velocity=0 -> lower=0 upper=0 effort=0 velocity=0
