Commit message: inserted chessboard_model

File: urdf/myCameraStereo.urdf (robot description, URDF)
Before this commit: robot myCameraStereo, 4 links, 3 joints
Links:
- removed link second_link
- removed link third_link
- added link horizontal_link, mass 0.01; collision box size=0.005 0.005 0.015; visual sphere radius=0.03
- added link horizontal_rotation_link, mass 0.01; collision box size=0.005 0.005 0.015; visual sphere radius=0.03
- added link vertical_link, mass 0.01; collision box size=0.005 0.005 0.015; visual sphere radius=0.03
- link cameras: mass 0.5 -> 0.01
Joints:
- removed joint base_to_second_joint
- removed joint base_to_third_joint
- added joint base_to_horizontal_link: type prismatic, parent horizontal_link, child horizontal_rotation_link, origin xyz=0 0 0.20 rpy=0 0 0, axis 0 1 0, limit lower=-1 upper=10 effort=100 velocity=1
- added joint base_to_horizontal_rotation_link: type revolute, parent horizontal_rotation_link, child cameras, origin xyz=0 0 0.10 rpy=0.0 0.0 0, axis 0 0 1, limit lower=-1 upper=10 effort=100 velocity=1
- added joint base_to_vertical_link: type prismatic, parent vertical_link, child horizontal_link, origin xyz=0 0 0.30 rpy=0 0 0, axis 1 0 0, limit lower=-1 upper=10 effort=100 velocity=1
- joint fixed_joint: axis 0 0 0 -> (none); child third_link -> vertical_link; limit lower=0 upper=0 effort=0 velocity=0 -> (none); type revolute -> fixed

Commit message: Removing gravity and installing yaml

File: urdf/myCameraStereo.urdf (robot description, URDF)
Before this commit: robot myCameraStereo, 5 links, 4 joints
Links:
- link vertical_link: mass 0.01 -> 1000
Joints:
- joint fixed_joint: axis (none) -> 0 0 1; limit (none) -> lower=0 upper=0 effort=20000 velocity=0; type fixed -> prismatic

Commit message: efforce correction model

File: urdf/myCameraStereo.urdf (robot description, URDF)
Before this commit: robot myCameraStereo, 5 links, 4 joints
Links:
- link cameras: mass 0.01 -> 1
- link horizontal_link: mass 0.01 -> 1
- link horizontal_rotation_link: mass 0.01 -> 1
- link vertical_link: mass 1000 -> 1
Joints:
- joint fixed_joint: limit lower=0 upper=0 effort=20000 velocity=0 -> lower=0 upper=3 effort=1000 velocity=0; type prismatic -> revolute

Commit message: correction pose robot

File: urdf/myCameraStereo.urdf (robot description, URDF)
Before this commit: robot myCameraStereo, 5 links, 4 joints
Joints:
- joint base_to_horizontal_link: origin xyz=0 0 0.20 rpy=0 0 0 -> xyz=0 0 0.10 rpy=0 0 0
- joint base_to_vertical_link: origin xyz=0 0 0.30 rpy=0 0 0 -> xyz=0 0 0.10 rpy=0 0 0
- joint fixed_joint: limit lower=0 upper=3 effort=1000 velocity=0 -> lower=0 upper=0 effort=1000 velocity=0

Commit message: Only chessboard world

File: urdf/myCameraStereo.urdf (robot description, URDF)
Before this commit: robot myCameraStereo, 5 links, 4 joints
Joints:
- joint base_to_horizontal_link: limit lower=-1 upper=10 effort=100 velocity=1 -> lower=-1 upper=10 effort=100 velocity=0.01
- joint base_to_horizontal_rotation_link: limit lower=-1 upper=10 effort=100 velocity=1 -> lower=-1 upper=10 effort=100 velocity=0.01
- joint base_to_vertical_link: limit lower=-1 upper=10 effort=100 velocity=1 -> lower=-1 upper=10 effort=100 velocity=0.01

Commit message: changes velocity, publish_frequency, ThDepth

File: urdf/myCameraStereo.urdf (robot description, URDF)
Before this commit: robot myCameraStereo, 5 links, 4 joints
Joints:
- joint base_to_horizontal_rotation_link: limit lower=-1 upper=10 effort=100 velocity=1 -> lower=-10 upper=10 effort=100 velocity=0.3
